File: tfk20/tfk20_regulator_usb_protection.sch (KiCad schematic (older format))
At the start: 14 parts, among them U3 TCCP01-M12, U4 MCP1700-3302E_SOT23, U5 USBLC6-2SC6

Commit message: Add STL11N3LLH6 footprint
Parts:
- gave numbers to parts that had none: 1
- renumbered C25 to C501, C26 to C502, C27 to C503, C28 to C504, D57 to D501, F1 to F501, R10 to R501, R11 to R502, R12 to R503, R13 to R504, U3 to U501, U4 to U502, U5 to U503
Other:
- note added: "Voltage regulator, USB VBUS/CC overvoltage/overcurrent and ESD protection"
- note removed: "Voltage regulator, USB VBUS/CC overvoltage and ESD protection"
Changed lines of the file:
@@
 $EndDescr
 $Comp
-L Regulator_Linear:MCP1700-3302E_SOT23 U4
+L Regulator_Linear:MCP1700-3302E_SOT23 U502
 U 1 1 6093AEA1
 P 5600 2950
-F 0 "U4" H 5600 3192 50  0000 C CNN
+F 0 "U502" H 5600 3192 50  0000 C CNN
 F 1 "MCP1700-3302E_SOT23" H 5600 3101 50  0000 C CNN
 F 2 "Package_TO_SOT_SMD:SOT-23" H 5600 3175 50  0001 C CNN
@@
 P 4900 2850
 AR Path="/6093AEA9" Ref="#PWR?"  Part="1"
-AR Path="/60815FFC/6093AEA9" Ref="#PWR053"  Part="1"
-F 0 "#PWR053" H 4900 2700 50  0001 C CNN
+AR Path="/60815FFC/6093AEA9" Ref="#PWR0504"  Part="1"
+F 0 "#PWR0504" H 4900 2700 50  0001 C CNN
 F 1 "+5V" H 4915 3023 50  0000 C CNN
 F 2 "" H 4900 2850 50  0001 C CNN
@@
 	6400 2950 6400 2850
 $Comp
-L power:+3.3V #PWR058
+L power:+3.3V #PWR0509
 U 1 1 6093AEB1
 P 6400 2850
-F 0 "#PWR058" H 6400 2700 50  0001 C CNN
+F 0 "#PWR0509" H 6400 2700 50  0001 C CNN
 F 1 "+3.3V" H 6415 3023 50  0000 C CNN
 F 2 "" H 6400 2850 50  0001 C CNN
@@
 $EndComp
 $Comp
-L power:GND #PWR056
+L power:GND #PWR0507
 U 1 1 6093AEB7
 P 5600 3250
-F 0 "#PWR056" H 5600 3000 50  0001 C CNN
+F 0 "#PWR0507" H 5600 3000 50  0001 C CNN
 F 1 "GND" H 5605 3077 50  0000 C CNN
 F 2 "" H 5600 3250 50  0001 C CNN
@@
 $EndComp
 $Comp
-L Device:C_Small C26
+L Device:C_Small C502
 U 1 1 6093AEBD
 P 5100 3100
-F 0 "C26" H 5192 3146 50  0000 L CNN
+F 0 "C502" H 5192 3146 50  0000 L CNN
 F 1 "1u" H 5192 3055 50  0000 L CNN
 F 2 "" H 5100 3100 50  0001 C CNN
@@
 $EndComp
 $Comp
-L power:GND #PWR055
+L power:GND #PWR0506
 U 1 1 6093AEC3
 P 5100 3250
-F 0 "#PWR055" H 5100 3000 50  0001 C CNN
+F 0 "#PWR0506" H 5100 3000 50  0001 C CNN
 F 1 "GND" H 5105 3077 50  0000 C CNN
 F 2 "" H 5100 3250 50  0001 C CNN
@@
 	5100 2950 5300 2950
 $Comp
-L Device:C_Small C27
+L Device:C_Small C503
 U 1 1 6093AECD
 P 6100 3100
-F 0 "C27" H 6192 3146 50  0000 L CNN
+F 0 "C503" H 6192 3146 50  0000 L CNN
 F 1 "1u" H 6192 3055 50  0000 L CNN
 F 2 "" H 6100 3100 50  0001 C CNN
@@
 $EndComp
 $Comp
-L power:GND #PWR057
+L power:GND #PWR0508
 U 1 1 6093AED3
 P 6100 3250
-F 0 "#PWR057" H 6100 3000 50  0001 C CNN
+F 0 "#PWR0508" H 6100 3000 50  0001 C CNN
 F 1 "GND" H 6105 3077 50  0000 C CNN
 F 2 "" H 6100 3250 50  0001 C CNN
@@
 P 2750 2950
 AR Path="/6093AEDF" Ref="F?"  Part="1"
-AR Path="/60815FFC/6093AEDF" Ref="F1"  Part="1"
-F 0 "F1" V 2545 2950 50  0000 C CNN
+AR Path="/60815FFC/6093AEDF" Ref="F501"  Part="1"
+F 0 "F501" V 2545 2950 50  0000 C CNN
 F 1 "500mA" V 2636 2950 50  0000 C CNN
 F 2 "" H 2800 2750 50  0001 L CNN
@@
 P 4400 4150
 AR Path="/6093AEE6" Ref="U?"  Part="1"
-AR Path="/60815FFC/6093AEE6" Ref="U3"  Part="1"
-F 0 "U3" H 4850 3400 50  0000 C CNN
+AR Path="/60815FFC/6093AEE6" Ref="U501"  Part="1"
+F 0 "U501" H 4850 3400 50  0000 C CNN
 F 1 "TCCP01-M12" H 4850 3300 50  0000 C CNN
 F 2 "Package_DFN_QFN:QFN-12-1EP_3x3mm_P0.5mm_EP1.65x1.65mm" H 4400 2800 50  0001 C CNN
@@
 P 3650 3500
 AR Path="/6093AEF2" Ref="C?"  Part="1"
-AR Path="/60815FFC/6093AEF2" Ref="C25"  Part="1"
-F 0 "C25" H 3742 3546 50  0000 L CNN
+AR Path="/60815FFC/6093AEF2" Ref="C501"  Part="1"
+F 0 "C501" H 3742 3546 50  0000 L CNN
 F 1 "100n" H 3742 3455 50  0000 L CNN
 F 2 "" H 3650 3500 50  0001 C CNN
@@
 P 3650 3600
 AR Path="/6093AEF8" Ref="#PWR?"  Part="1"
-AR Path="/60815FFC/6093AEF8" Ref="#PWR051"  Part="1"
-F 0 "#PWR051" H 3650 3350 50  0001 C CNN
+AR Path="/60815FFC/6093AEF8" Ref="#PWR0502"  Part="1"
+F 0 "#PWR0502" H 3650 3350 50  0001 C CNN
 F 1 "GND" H 3655 3427 50  0000 C CNN
 F 2 "" H 3650 3600 50  0001 C CNN
@@
 P 3050 4200
 AR Path="/6093AEFF" Ref="R?"  Part="1"
-AR Path="/60815FFC/6093AEFF" Ref="R11"  Part="1"
-F 0 "R11" H 3109 4246 50  0000 L CNN
+AR Path="/60815FFC/6093AEFF" Ref="R502"  Part="1"
+F 0 "R502" H 3109 4246 50  0000 L CNN
 F 1 "2.7k" H 3109 4155 50  0000 L CNN
 F 2 "" H 3050 4200 50  0001 C CNN
@@
 P 3050 4300
 AR Path="/6093AF08" Ref="#PWR?"  Part="1"
-AR Path="/60815FFC/6093AF08" Ref="#PWR050"  Part="1"
-F 0 "#PWR050" H 3050 4050 50  0001 C CNN
+AR Path="/60815FFC/6093AF08" Ref="#PWR0501"  Part="1"
+F 0 "#PWR0501" H 3050 4050 50  0001 C CNN
 F 1 "GND" H 3055 4127 50  0000 C CNN
 F 2 "" H 3050 4300 50  0001 C CNN
@@
 P 3050 3800
 AR Path="/6093AF0E" Ref="R?"  Part="1"
-AR Path="/60815FFC/6093AF0E" Ref="R10"  Part="1"
-F 0 "R10" H 3109 3846 50  0000 L CNN
+AR Path="/60815FFC/6093AF0E" Ref="R501"  Part="1"
+F 0 "R501" H 3109 3846 50  0000 L CNN
 F 1 "10k" H 3109 3755 50  0000 L CNN
 F 2 "" H 3050 3800 50  0001 C CNN
@@
 	3650 3400 3650 3350
 Wire Wire Line
-	3650 3350 3450 3350
-Wire Wire Line
-	4300 3450 4300 3350
-Wire Wire Line
-	4300 3350 3650 3350
-Connection ~ 3650 3350
-Wire Wire Line
-	3250 3350 3050 3350
-Wire Wire Line
-	3050 3350 3050 3700
-Wire Wire Line
 	3900 4350 3850 4350
 Wire Wire Line
@@
 P 5000 4500
 AR Path="/6093AF1F" Ref="#PWR?"  Part="1"
-AR Path="/60815FFC/6093AF1F" Ref="#PWR054"  Part="1"
-F 0 "#PWR054" H 5000 4250 50  0001 C CNN
+AR Path="/60815FFC/6093AF1F" Ref="#PWR0505"  Part="1"
+F 0 "#PWR0505" H 5000 4250 50  0001 C CNN
 F 1 "GND" H 5005 4327 50  0000 C CNN
 F 2 "" H 5000 4500 50  0001 C CNN
@@
 P 4400 4950
 AR Path="/6093AF37" Ref="#PWR?"  Part="1"
-AR Path="/60815FFC/6093AF37" Ref="#PWR052"  Part="1"
-F 0 "#PWR052" H 4400 4700 50  0001 C CNN
+AR Path="/60815FFC/6093AF37" Ref="#PWR0503"  Part="1"
+F 0 "#PWR0503" H 4400 4700 50  0001 C CNN
 F 1 "GND" H 4405 4777 50  0000 C CNN
 F 2 "" H 4400 4950 50  0001 C CNN
@@
 $EndComp
 Wire Wire Line
-	3050 2950 2850 2950
-Wire Wire Line
-	2650 2950 2500 2950
-Wire Wire Line
 	4500 3450 4500 3350
 Wire Wire Line
@@
 VBUS OVP\nset to 6V
 Wire Wire Line
-	3050 2950 3050 3350
-Connection ~ 3050 3350
-Wire Wire Line
 	4700 3350 4700 2950
 Connection ~ 4700 2950
 Wire Wire Line
 	4600 2950 4700 2950
-Wire Wire Line
-	4200 2950 3050 2950
-Connection ~ 3050 2950
 Text Notes 3550 2650 0    50   ~ 0
 TODO: Update MOSFET\nfootprint
@@
 	4700 2950 4900 2950
 Text Notes 2200 2400 0    50   ~ 0
-Voltage regulator, USB VBUS/CC overvoltage and ESD protection
+Voltage regulator, USB VBUS/CC overvoltage/overcurrent and ESD protection
 Wire Notes Line
 	2150 2250 2150 5250
@@
 P 8950 4000
 AR Path="/6093F36B" Ref="C?"  Part="1"
-AR Path="/60815FFC/6093F36B" Ref="C28"  Part="1"
-F 0 "C28" H 9200 3950 50  0000 R CNN
+AR Path="/60815FFC/6093F36B" Ref="C504"  Part="1"
+F 0 "C504" H 9200 3950 50  0000 R CNN
 F 1 "4.7n" H 9200 4050 50  0000 R CNN
 F 2 "" H 8950 4000 50  0001 C CNN
@@
 P 8950 4100
 AR Path="/6093F371" Ref="#PWR?"  Part="1"
-AR Path="/60815FFC/6093F371" Ref="#PWR060"  Part="1"
-F 0 "#PWR060" H 8950 3850 50  0001 C CNN
+AR Path="/60815FFC/6093F371" Ref="#PWR0511"  Part="1"
+F 0 "#PWR0511" H 8950 3850 50  0001 C CNN
 F 1 "GND" H 8955 3927 50  0000 C CNN
 F 2 "" H 8950 4100 50  0001 C CNN
@@
 P 7800 3800
 AR Path="/6093F37C" Ref="U?"  Part="1"
-AR Path="/60815FFC/6093F37C" Ref="U5"  Part="1"
-F 0 "U5" V 7500 4400 50  0000 C CNN
+AR Path="/60815FFC/6093F37C" Ref="U503"  Part="1"
+F 0 "U503" V 7500 4400 50  0000 C CNN
 F 1 "USBLC6-2SC6" V 7600 4400 50  0000 C CNN
 F 2 "Package_TO_SOT_SMD:SOT-23-6" H 7800 3300 50  0001 C CNN
@@
 P 8100 3300
 AR Path="/6093F386" Ref="R?"  Part="1"
-AR Path="/60815FFC/6093F386" Ref="R12"  Part="1"
-F 0 "R12" V 7904 3300 50  0000 C CNN
+AR Path="/60815FFC/6093F386" Ref="R503"  Part="1"
+F 0 "R503" V 7904 3300 50  0000 C CNN
 F 1 "22" V 7995 3300 50  0000 C CNN
 F 2 "" H 8100 3300 50  0001 C CNN
@@
 P 8100 4300
 AR Path="/6093F38F" Ref="R?"  Part="1"
-AR Path="/60815FFC/6093F38F" Ref="R13"  Part="1"
-F 0 "R13" V 8200 4300 50  0000 C CNN
+AR Path="/60815FFC/6093F38F" Ref="R504"  Part="1"
+F 0 "R504" V 8200 4300 50  0000 C CNN
 F 1 "22" V 8300 4300 50  0000 C CNN
 F 2 "" H 8100 4300 50  0001 C CNN
@@
 P 7300 3900
 AR Path="/6093F3A1" Ref="#PWR?"  Part="1"
-AR Path="/60815FFC/6093F3A1" Ref="#PWR059"  Part="1"
-F 0 "#PWR059" H 7300 3650 50  0001 C CNN
+AR Path="/60815FFC/6093F3A1" Ref="#PWR0510"  Part="1"
+F 0 "#PWR0510" H 7300 3650 50  0001 C CNN
 F 1 "GND" H 7305 3727 50  0000 C CNN
 F 2 "" H 7300 3900 50  0001 C CNN
@@
 P 9150 3700
 AR Path="/6093F3AA" Ref="#PWR?"  Part="1"
-AR Path="/60815FFC/6093F3AA" Ref="#PWR061"  Part="1"
-F 0 "#PWR061" H 9150 3550 50  0001 C CNN
+AR Path="/60815FFC/6093F3AA" Ref="#PWR0512"  Part="1"
+F 0 "#PWR0512" H 9150 3550 50  0001 C CNN
 F 1 "+5V" H 9165 3873 50  0000 C CNN
 F 2 "" H 9150 3700 50  0001 C CNN
@@
 P 3350 3350
 AR Path="/6093AEEC" Ref="D?"  Part="1"
-AR Path="/60815FFC/6093AEEC" Ref="D57"  Part="1"
-F 0 "D57" H 3350 3143 50  0000 C CNN
+AR Path="/60815FFC/6093AEEC" Ref="D501"  Part="1"
+F 0 "D501" H 3350 3143 50  0000 C CNN
 F 1 "D_Schottky_Small" H 3350 3234 50  0000 C CNN
 F 2 "" V 3350 3350 50  0001 C CNN
@@
 $EndComp
 $Comp
-L tfk:STL11N3LLH6 Q?
+L tfk:STL11N3LLH6 Q501
 U 1 1 603EB8D8
 P 4400 3050
-F 0 "Q?" V 4742 3050 50  0000 C CNN
+F 0 "Q501" V 4742 3050 50  0000 C CNN
 F 1 "STL11N3LLH6" V 4651 3050 50  0000 C CNN
 F 2 "Package_TO_SOT_SMD:LFPAK33" H 4600 2975 50  0001 L CIN
@@
 	0    -1   -1   0
 $EndComp
+Wire Wire Line
+	3050 2950 3050 3350
+Connection ~ 3050 2950
+Connection ~ 3050 3350
+Wire Wire Line
+	3050 3350 3050 3700
+Connection ~ 3650 3350
+Wire Wire Line
+	4300 3350 4300 3450
+Wire Wire Line
+	2500 2950 2650 2950
+Wire Wire Line
+	2850 2950 3050 2950
+Wire Wire Line
+	3050 2950 4200 2950
+Wire Wire Line
+	3050 3350 3250 3350
+Wire Wire Line
+	3450 3350 3650 3350
+Wire Wire Line
+	3650 3350 4300 3350
 $EndSCHEMATC

Commit message: Fix project
Parts:
- Q501: footprint Package_TO_SOT_SMD:LFPAK33 -> STL11N3LLH6:STL11N3LLH6
- U501: footprint Package_DFN_QFN:QFN-12-1EP_3x3mm_P0.5mm_EP1.65x1.65mm -> Package_DFN_QFN:QFN-12-1EP_3x3mm_P0.51mm_EP1.45x1.45mm
Changed lines of the file:
@@
 Connection ~ 4900 2950
-$Comp
-L tfk:TCCP01-M12 U?
-U 1 1 6093AEE6
-P 4400 4150
-AR Path="/6093AEE6" Ref="U?"  Part="1"
-AR Path="/60815FFC/6093AEE6" Ref="U501"  Part="1"
-F 0 "U501" H 4850 3400 50  0000 C CNN
-F 1 "TCCP01-M12" H 4850 3300 50  0000 C CNN
-F 2 "Package_DFN_QFN:QFN-12-1EP_3x3mm_P0.5mm_EP1.65x1.65mm" H 4400 2800 50  0001 C CNN
-F 3 "https://www.st.com/resource/en/datasheet/tcpp01-m12.pdf" H 4250 4450 50  0001 C CNN
-	1    4400 4150
-	1    0    0    -1
-$EndComp
 $Comp
 L Device:C_Small C?
@@
 	-1   0    0    1
 $EndComp
+Wire Wire Line
+	3050 2950 3050 3350
+Connection ~ 3050 2950
+Connection ~ 3050 3350
+Wire Wire Line
+	3050 3350 3050 3700
+Connection ~ 3650 3350
+Wire Wire Line
+	4300 3350 4300 3450
+Wire Wire Line
+	2500 2950 2650 2950
+Wire Wire Line
+	2850 2950 3050 2950
+Wire Wire Line
+	3050 2950 4200 2950
+Wire Wire Line
+	3050 3350 3250 3350
+Wire Wire Line
+	3450 3350 3650 3350
+Wire Wire Line
+	3650 3350 4300 3350
+$Comp
+L tfk:TCCP01-M12 U501
+U 1 1 60432DBC
+P 4400 4150
+F 0 "U501" H 4800 3450 50  0000 C CNN
+F 1 "TCCP01-M12" H 4800 3350 50  0000 C CNN
+F 2 "Package_DFN_QFN:QFN-12-1EP_3x3mm_P0.51mm_EP1.45x1.45mm" H 4400 3050 50  0001 C CNN
+F 3 "https://www.st.com/resource/en/datasheet/tcpp01-m12.pdf" H 4350 4300 50  0001 C CNN
+	1    4400 4150
+	1    0    0    -1
+$EndComp
 $Comp
 L tfk:STL11N3LLH6 Q501
-U 1 1 603EB8D8
+U 1 1 60434876
 P 4400 3050
 F 0 "Q501" V 4742 3050 50  0000 C CNN
 F 1 "STL11N3LLH6" V 4651 3050 50  0000 C CNN
-F 2 "Package_TO_SOT_SMD:LFPAK33" H 4600 2975 50  0001 L CIN
-F 3 "https://assets.nexperia.com/documents/data-sheet/BUK9M53-60E.pdf" V 4400 3050 50  0001 L CNN
+F 2 "STL11N3LLH6:STL11N3LLH6" H 4600 2975 50  0001 L CIN
+F 3 "https://www.st.com/resource/en/datasheet/stl11n3llh6.pdf" V 4400 3050 50  0001 L CNN
 	1    4400 3050
 	0    -1   -1   0
 $EndComp
-Wire Wire Line
-	3050 2950 3050 3350
-Connection ~ 3050 2950
-Connection ~ 3050 3350
-Wire Wire Line
-	3050 3350 3050 3700
-Connection ~ 3650 3350
-Wire Wire Line
-	4300 3350 4300 3450
-Wire Wire Line
-	2500 2950 2650 2950
-Wire Wire Line
-	2850 2950 3050 2950
-Wire Wire Line
-	3050 2950 4200 2950
-Wire Wire Line
-	3050 3350 3250 3350
-Wire Wire Line
-	3450 3350 3650 3350
-Wire Wire Line
-	3650 3350 4300 3350
 $EndSCHEMATC
