File: tfk20-avr/tfk20-avr.kicad_pcb (KiCad board)
At the start: 4 copper layers, 76.2 x 115.5 mm, 123 parts, among them J1 USB_C_Receptacle_USB2.0, J2 AVR-ISP-6, SW1 Reset, U1 ATmega32U4-AU, U2 IS31FL3733-TQ, Y1 16MHz

Commit message: Continue routing
Connections:
- U1 pad 40: /ROW_4 -> /ROW_5
- U1 pad 41: /ROW_5 -> /ROW_4
Routing:
- net /ROW_5: track 0.00 -> 91.2 mm, vias 0 -> 3
- net /ROW_0: track 4.17 -> 68.2 mm
- net /ROW_4: track 0.00 -> 62.6 mm, vias 0 -> 4
- net /ROW_1: track 0.00 -> 58.0 mm, vias 0 -> 5
- net /ROW_3: track 0.00 -> 48.1 mm, vias 0 -> 4
- net /ROW_2: track 0.00 -> 43.6 mm, vias 0 -> 4
- net /RGB_MATRIX_SCL: track 0.00 -> 32.4 mm, vias 0 -> 2
- net /RGB_MATRIX_SDA: track 0.00 -> 29.8 mm, vias 0 -> 2
- net Net-(D18-Pad2): track 0.00 -> 29.7 mm, vias 0 -> 2
- net /MISO: track 0.00 -> 27.4 mm, vias 0 -> 1
- net /MOSI: track 0.00 -> 25.8 mm, vias 0 -> 1
- net /SCK: track 0.00 -> 24.3 mm, vias 0 -> 1
- net /RGB_LIGHT: track 0.00 -> 17.0 mm, vias 0 -> 2
- net /RESET: track 3.48 -> 8.22 mm, vias 1 -> 2

Commit message: Continue routing
Connections:
- U1 pad 27: /COL_2 -> /COL_3
- U1 pad 28: /COL_1 -> /COL_2
- U1 pad 29: /COL_0 -> /COL_1
- U1 pad 30: /COL_3 -> /RGB_LIGHT
- U1 pad 31: /RGB_LIGHT -> /COL_0
Routing:
- net /COL_0: track 107.8 -> 181.7 mm, vias 0 -> 2
- net /RESET: track 8.22 -> 62.7 mm, vias 2 -> 3
- net /COL_1: track 77.7 -> 125.3 mm, vias 2 -> 4
- net /COL_2: track 79.2 -> 125.1 mm, vias 0 -> 4
- net /SCK: track 24.3 -> 54.3 mm, vias 1 -> 2
- net Net-(D18-Pad2): track 29.7 -> 0.00 mm, vias 2 -> 0
- net /MOSI: track 25.8 -> 51.6 mm, vias 1 -> 2
- net /ROW_3: track 48.1 -> 73.6 mm
- net /MISO: track 27.4 -> 51.9 mm, vias 1 -> 2
- net /ROW_1: track 58.0 -> 82.4 mm
- net /ROW_2: track 43.6 -> 65.3 mm
- net /ROW_0: track 68.2 -> 88.4 mm
- net /COL_3: track 39.9 -> 41.1 mm, vias 0 -> 1
- net /ROW_5: track 91.2 -> 92.0 mm
- net /RGB_LIGHT: track 17.0 -> 17.6 mm

Commit message: Continue routing
Parts:
- moved C4 0.51 mm to (177.3, 124.5)
Routing:
- net /tfk20 RGB Matrix/SW5: track 0.00 -> 157.8 mm, vias 0 -> 8
- net /tfk20 RGB Matrix/SW4: track 0.00 -> 139.0 mm, vias 0 -> 8
- net /RESET: track 62.7 -> 144.7 mm, vias 3 -> 5
- net /tfk20 RGB Matrix/SW6: track 0.00 -> 81.9 mm, vias 0 -> 6
- net /SHIELD: track 0.00 -> 51.6 mm
- net /tfk20 RGB Matrix/SW7: track 0.00 -> 50.9 mm, vias 0 -> 3
- net /ROW_0: track 88.4 -> 138.5 mm, vias 4 -> 5
- net /tfk20 RGB Matrix/SW8: track 0.00 -> 48.6 mm, vias 0 -> 3
- net /COL_3: track 41.1 -> 86.8 mm, vias 1 -> 3
- net /tfk20 RGB Matrix/CS5: track 0.00 -> 45.0 mm, vias 0 -> 2
- net /ROW_1: track 82.4 -> 120.5 mm
- net Net-(R7-Pad2): track 0.00 -> 29.2 mm
- net /ROW_2: track 65.3 -> 84.8 mm, vias 4 -> 5
- net Net-(D3-Pad2): track 0.00 -> 9.96 mm
- net Net-(C8-Pad1): track 0.00 -> 4.50 mm
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
Commit message: Continue routing
Connections:
- U2 pad 10: /tfk20 RGB Matrix/SW8 -> /tfk20 RGB Matrix/SW2
- U2 pad 11: /tfk20 RGB Matrix/SW9 -> /tfk20 RGB Matrix/SW3
- U2 pad 2: /tfk20 RGB Matrix/SW1 -> /tfk20 RGB Matrix/SW7
- U2 pad 3: /tfk20 RGB Matrix/SW2 -> /tfk20 RGB Matrix/SW8
- U2 pad 4: /tfk20 RGB Matrix/SW3 -> /tfk20 RGB Matrix/SW9
- U2 pad 9: /tfk20 RGB Matrix/SW7 -> /tfk20 RGB Matrix/SW1
Routing:
- net /tfk20 RGB Matrix/SW2: track 0.00 -> 177.0 mm, vias 0 -> 11
- net /tfk20 RGB Matrix/SW9: track 0.00 -> 175.9 mm, vias 0 -> 13
- net /tfk20 RGB Matrix/SW3: track 0.00 -> 169.5 mm, vias 0 -> 9
- net /tfk20 RGB Matrix/SW1: track 0.00 -> 167.5 mm, vias 0 -> 9
- net /tfk20 RGB Matrix/SW7: track 50.9 -> 196.7 mm, vias 3 -> 11
- net /tfk20 RGB Matrix/CS1: track 0.00 -> 145.6 mm, vias 0 -> 4
- net /tfk20 RGB Matrix/SW8: track 48.6 -> 188.4 mm, vias 3 -> 11
- net /tfk20 RGB Matrix/CS3: track 0.00 -> 129.6 mm, vias 0 -> 6
- net /tfk20 RGB Matrix/CS2: track 0.00 -> 127.1 mm, vias 0 -> 4
- net /tfk20 RGB Matrix/CS8: track 0.00 -> 115.3 mm, vias 0 -> 8
- net /tfk20 RGB Matrix/CS5: track 45.0 -> 157.8 mm, vias 2 -> 3
- net /tfk20 RGB Matrix/CS6: track 0.00 -> 89.5 mm, vias 0 -> 2
- net /tfk20 RGB Matrix/CS7: track 0.00 -> 68.5 mm, vias 0 -> 2
- net /tfk20 RGB Matrix/SW6: track 81.9 -> 133.3 mm, vias 6 -> 10
- net /tfk20 RGB Matrix/CS4: track 0.00 -> 38.5 mm
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
Commit message: Finish routing
Routing:
- net /tfk20 RGB Matrix/CS7: track 68.5 -> 127.6 mm, vias 2 -> 4
- net Net-(D25-Pad2): track 0.00 -> 48.2 mm, vias 0 -> 2
- net Net-(D28-Pad2): track 0.00 -> 40.4 mm, vias 0 -> 2
- net Net-(D26-Pad2): track 0.00 -> 26.1 mm
- net Net-(D29-Pad2): track 0.00 -> 26.0 mm, vias 0 -> 2
- net Net-(D27-Pad2): track 0.00 -> 19.7 mm, vias 0 -> 2
- net /tfk20 RGB Matrix/SW8: track 188.4 -> 182.4 mm
- net /tfk20 RGB Matrix/SW7: track 196.7 -> 198.8 mm, vias 11 -> 10
- net /COL_1: track 127.8 -> 129.8 mm
- net /tfk20 RGB Matrix/SW9: track 175.9 -> 177.4 mm
- net /tfk20 RGB Matrix/SW2: track 177.0 -> 175.9 mm
- net /tfk20 RGB Matrix/SW3: track 169.5 -> 168.4 mm
- net /tfk20 RGB Matrix/SW1: track 167.5 -> 166.4 mm
- net GND: track 126.5 -> 127.2 mm

Commit message: Tweak some routes
Routing:
- net /COL_2: track 126.4 -> 127.6 mm
- net GND: track 127.2 -> 126.4 mm
Other:
- board text added: "Rev. A"
- board text removed: "Rev. 0"
Changed lines of the file:
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@@
     (thickness 1.6)
     (drawings 36)
-    (tracks 1694)
+    (tracks 1697)
     (zones 0)
     (modules 123)
@@
     (title tfk20-avr)
     (date 2021-06-12)
-    (rev 0)
+    (rev A)
     (company biosmanager)
   )
@@
     (34 B.Paste user)
     (35 F.Paste user)
-    (36 B.SilkS user hide)
-    (37 F.SilkS user hide)
+    (36 B.SilkS user)
+    (37 F.SilkS user)
     (38 B.Mask user)
     (39 F.Mask user)
@@
     )
   )
-  (gr_text "Rev. 0" (at 176.609375 150.01875) (layer B.SilkS)
+  (gr_text "Rev. A" (at 170.65625 150.8125) (layer B.SilkS)
     (effects (font (size 1 1) (thickness 0.15)) (justify mirror))
   )
@@
   (segment (start 164.375 95.2375) (end 164.375 94.07) (width 0.381) (layer B.Cu) (net 1) (status 10))
   (segment (start 165.227 93.218) (end 165.227 91.4615) (width 0.381) (layer B.Cu) (net 1) (status 20))
-  (segment (start 171.323 101.9595) (end 172.6985 101.9595) (width 0.381) (layer B.Cu) (net 1) (status 10))
   (via (at 173.101 103.759) (size 0.8) (drill 0.4) (layers F.Cu B.Cu) (net 1))
-  (segment (start 173.101 102.362) (end 173.101 103.759) (width 0.381) (layer B.Cu) (net 1))
-  (segment (start 172.6985 101.9595) (end 173.101 102.362) (width 0.381) (layer B.Cu) (net 1))
   (segment (start 174.9845 104.521) (end 173.482 104.521) (width 0.381) (layer B.Cu) (net 1) (status 10))
   (segment (start 174.9845 104.521) (end 173.228 104.521) (width 0.381) (layer B.Cu) (net 1) (status 10))
@@
   (segment (start 170.725 126.289) (end 169.3166 126.289) (width 0.381) (layer B.Cu) (net 1) (status 10))
   (via (at 169.3164 126.2888) (size 0.8) (drill 0.4) (layers F.Cu B.Cu) (net 1))
+  (segment (start 171.323 101.981) (end 173.101 103.759) (width 0.381) (layer B.Cu) (net 1))
+  (segment (start 171.323 101.9595) (end 171.323 101.981) (width 0.381) (layer B.Cu) (net 1))
   (via (at 147.0152 62.5348) (size 0.8) (drill 0.4) (layers F.Cu B.Cu) (net 2))
   (segment (start 147.023 62.527) (end 147.0152 62.5348) (width 0.381) (layer B.Cu) (net 2))
@@
   (segment (start 165.4302 74.2188) (end 167.767006 74.2188) (width 0.254) (layer F.Cu) (net 50))
   (segment (start 154.305 75.692002) (end 155.086003 74.910999) (width 0.254) (layer F.Cu) (net 50))
-  (segment (start 169.955439 68.579425) (end 173.224 71.847986) (width 0.254) (layer B.Cu) (net 51))
+  (segment (start 173.224 71.847986) (end 173.224 76.3555) (width 0.254) (layer B.Cu) (net 51))
   (segment (start 169.955439 61.371639) (end 169.955439 68.579425) (width 0.254) (layer B.Cu) (net 51))
-  (segment (start 173.070651 52.644637) (end 173.070651 58.256427) (width 0.254) (layer B.Cu) (net 51))
-  (segment (start 170.2816 49.855586) (end 173.070651 52.644637) (width 0.254) (layer B.Cu) (net 51))
-  (segment (start 173.070651 58.256427) (end 169.955439 61.371639) (width 0.254) (layer B.Cu) (net 51))
-  (segment (start 170.2816 42.6944) (end 170.2816 49.855586) (width 0.254) (layer B.Cu) (net 51))
-  (segment (start 173.224 71.847986) (end 173.224 76.3555) (width 0.254) (layer B.Cu) (net 51) (status 20))
+  (segment (start 169.955439 68.579425) (end 173.224 71.847986) (width 0.254) (layer B.Cu) (net 51))
+  (segment (start 170.2816 49.1236) (end 173.5582 52.4002) (width 0.254) (layer B.Cu) (net 51))
+  (segment (start 173.5582 52.4002) (end 173.5582 57.768878) (width 0.254) (layer B.Cu) (net 51))
   (segment (start 170.38725 42.58875) (end 170.2816 42.6944) (width 0.254) (layer B.Cu) (net 51))
-  (segment (start 171.23625 42.58875) (end 170.38725 42.58875) (width 0.254) (layer B.Cu) (net 51) (status 10))
+  (segment (start 173.5582 57.768878) (end 169.955439 61.371639) (width 0.254) (layer B.Cu) (net 51))
+  (segment (start 170.2816 42.6944) (end 170.2816 49.1236) (width 0.254) (layer B.Cu) (net 51))
+  (segment (start 171.23625 42.58875) (end 170.38725 42.58875) (width 0.254) (layer B.Cu) (net 51))
   (via (at 112.649 84.328) (size 0.6) (drill 0.3) (layers F.Cu B.Cu) (net 52))
   (segment (start 112.649 77.399886) (end 112.649 84.328) (width 0.254) (layer F.Cu) (net 52))
@@
   (segment (start 180.071 115.09375) (end 177.89525 115.09375) (width 0.254) (layer B.Cu) (net 72) (status 10))
   (via (at 177.419 115.57) (size 0.6) (drill 0.3) (layers F.Cu B.Cu) (net 72))
-  (segment (start 162.1282 89.3207) (end 161.86625 89.05875) (width 0.254) (layer B.Cu) (net 72) (status 30))
-  (segment (start 162.1282 107.8468) (end 162.1282 89.3207) (width 0.254) (layer B.Cu) (net 72) (status 30))
-  (segment (start 161.86625 108.10875) (end 162.1282 107.8468) (width 0.254) (layer B.Cu) (net 72) (status 30))
   (segment (start 160.1724 109.8296) (end 160.1724 113.5634) (width 0.254) (layer B.Cu) (net 72))
   (segment (start 161.925 108.077) (end 160.1724 109.8296) (width 0.254) (layer B.Cu) (net 72) (status 10))
@@
   (segment (start 176.784 120.142) (end 169.799 127.127) (width 0.254) (layer F.Cu) (net 72))
   (segment (start 169.799 127.127) (end 168.325812 127.127) (width 0.254) (layer F.Cu) (net 72))
+  (segment (start 162.1282 105.7402) (end 162.1282 107.8468) (width 0.254) (layer B.Cu) (net 72))
+  (segment (start 160.7058 104.3178) (end 162.1282 105.7402) (width 0.254) (layer B.Cu) (net 72))
+  (segment (start 162.1282 107.8468) (end 161.86625 108.10875) (width 0.254) (layer B.Cu) (net 72))
+  (segment (start 160.7058 101.981) (end 160.7058 104.3178) (width 0.254) (layer B.Cu) (net 72))
+  (segment (start 162.1282 100.5586) (end 160.7058 101.981) (width 0.254) (layer B.Cu) (net 72))
+  (segment (start 162.1282 89.3207) (end 162.1282 100.5586) (width 0.254) (layer B.Cu) (net 72))
+  (segment (start 161.86625 89.05875) (end 162.1282 89.3207) (width 0.254) (layer B.Cu) (net 72))
   (segment (start 180.91625 50.95875) (end 180.91625 70.00875) (width 0.254) (layer B.Cu) (net 73) (status 30))
   (segment (start 176.37125 85.67045) (end 180.086 81.9557) (width 0.254) (layer B.Cu) (net 73))

Commit message: Fix silkscreen
Parts:
- moved R7 1.99 mm to (175.8, 146.9), turned to 0 degrees
Routing:
- net Net-(R7-Pad2): track 29.2 -> 30.9 mm

Commit message: Place OVP diode after fuse
Parts:
- moved F1 3.21 mm to (124.6, 64.3)
- moved D1 3.14 mm to (127.8, 64.3), turned to 90 degrees
Connections:
- D1 pad 1: VBUS -> +5V
Routing:
- net +5V: track 105.1 -> 108.5 mm
- net VBUS: track 32.9 -> 29.7 mm
Changed lines of the file:
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@@
     (thickness 1.6)
     (drawings 36)
-    (tracks 1696)
+    (tracks 1700)
     (zones 0)
     (modules 123)
@@
   )
   (module Fuse:Fuse_1206_3216Metric_Pad1.42x1.75mm_HandSolder (layer B.Cu)
-    (at 127.79375 64.29375 90)
+    (at 124.587 64.262 90)
     (descr "Fuse SMD 1206 (3216 Metric), square (rectangular) end terminal, IPC_7351 nominal with elongated pad for handsoldering. (Body size source: http://www.tortai-tech.com/upload/download/2011102023233369053.pdf), generated with kicad-footprint-generator")
     (tags "fuse handsolder")
     (attr smd)
-    (fp_text reference F1 (at 0.03175 2.12725 90) (layer B.SilkS)
+    (fp_text reference F1 (at 0 -1.778 90) (layer B.SilkS)
       (effects (font (size 1 1) (thickness 0.15)) (justify mirror))
     )
@@
   )
   (module Diode_SMD:D_SOD-123 (layer B.Cu)
-    (at 124.61875 64.29375 270)
+    (at 127.762 64.262 90)
     (descr SOD-123)
     (tags SOD-123)
     (attr smd)
-    (fp_text reference D1 (at 0 2 90) (layer B.SilkS)
+    (fp_text reference D1 (at 0 2.032 90) (layer B.SilkS)
       (effects (font (size 1 1) (thickness 0.15)) (justify mirror))
     )
@@
       (effects (font (size 1 1) (thickness 0.15)) (justify mirror))
     )
-    (pad 1 smd rect (at -1.65 0 270) (size 0.9 1.2) (layers B.Cu B.Paste B.Mask)
-      (net 105 VBUS))
-    (pad 2 smd rect (at 1.65 0 270) (size 0.9 1.2) (layers B.Cu B.Paste B.Mask)
+    (pad 1 smd rect (at -1.65 0 90) (size 0.9 1.2) (layers B.Cu B.Paste B.Mask)
+      (net 2 +5V))
+    (pad 2 smd rect (at 1.65 0 90) (size 0.9 1.2) (layers B.Cu B.Paste B.Mask)
       (net 1 GND))
     (model ${KISYS3DMOD}/Diode_SMD.3dshapes/D_SOD-123.wrl
@@
   (segment (start 163.5506 110.4861) (end 163.5506 109.8296) (width 0.381) (layer B.Cu) (net 1))
   (segment (start 164.3165 111.252) (end 163.5506 110.4861) (width 0.381) (layer B.Cu) (net 1) (status 10))
-  (via (at 124.61875 67.157606) (size 0.8) (drill 0.4) (layers F.Cu B.Cu) (net 1))
-  (segment (start 124.61875 65.94375) (end 124.61875 67.157606) (width 0.381) (layer B.Cu) (net 1) (status 10))
+  (via (at 124.61875 67.157606) (size 0.8) (drill 0.4) (layers F.Cu B.Cu) (net 2))
   (via (at 121.031 44.73579) (size 0.8) (drill 0.4) (layers F.Cu B.Cu) (net 1))
   (segment (start 129.059375 44.129375) (end 129.66579 44.73579) (width 0.381) (layer B.Cu) (net 1) (status 10))
@@
   (segment (start 125.34375 122.25) (end 125.34375 120.65525) (width 0.381) (layer B.Cu) (net 2) (status 10))
   (via (at 125.349 120.65) (size 0.8) (drill 0.4) (layers F.Cu B.Cu) (net 2))
-  (via (at 127.793749 67.1576) (size 0.8) (drill 0.4) (layers F.Cu B.Cu) (net 2))
-  (segment (start 127.79375 65.78125) (end 127.793749 66.591915) (width 0.381) (layer B.Cu) (net 2) (status 10))
-  (segment (start 127.793749 66.591915) (end 127.793749 67.1576) (width 0.381) (layer B.Cu) (net 2))
+  (via (at 129.286 62.611) (size 0.8) (drill 0.4) (layers F.Cu B.Cu) (net 1))
+  (segment (start 127.763 62.611) (end 127.762 62.612) (width 0.381) (layer B.Cu) (net 1))
+  (segment (start 129.286 62.611) (end 127.763 62.611) (width 0.381) (layer B.Cu) (net 1))
   (via (at 124.714 76.938201) (size 0.8) (drill 0.4) (layers F.Cu B.Cu) (net 2))
   (segment (start 123.317 78.335201) (end 124.714 76.938201) (width 0.381) (layer B.Cu) (net 2) (status 10))
@@
   (segment (start 168.3219 76.327) (end 166.9796 74.9847) (width 0.381) (layer B.Cu) (net 2) (status 10))
   (segment (start 166.9796 74.9847) (end 166.9796 74.980798) (width 0.381) (layer B.Cu) (net 2))
+  (segment (start 124.587 67.125856) (end 124.61875 67.157606) (width 0.381) (layer B.Cu) (net 2))
+  (segment (start 124.6245 65.7495) (end 124.587 65.7495) (width 0.381) (layer B.Cu) (net 2))
+  (segment (start 124.7495 65.912) (end 124.587 65.7495) (width 0.381) (layer B.Cu) (net 2))
+  (segment (start 127.762 65.912) (end 124.7495 65.912) (width 0.381) (layer B.Cu) (net 2))
+  (segment (start 124.61875 65.78125) (end 124.587 65.7495) (width 0.381) (layer B.Cu) (net 2))
+  (segment (start 124.61875 67.157606) (end 124.61875 65.78125) (width 0.381) (layer B.Cu) (net 2))
   (segment (start 130.129375 39.034375) (end 130.129375 43.214375) (width 0.254) (layer B.Cu) (net 3) (status 30))
   (segment (start 130.129375 39.034375) (end 121.489375 39.034375) (width 0.254) (layer B.Cu) (net 3) (status 30))
@@
   (segment (start 159.69459 129.921) (end 162.941 129.921) (width 0.254) (layer F.Cu) (net 69))
   (segment (start 158.142792 131.472798) (end 159.69459 129.921) (width 0.254) (layer F.Cu) (net 69))
-  (segment (start 123.76625 67.25125) (end 123.76625 70.00875) (width 0.254) (layer B.Cu) (net 70) (status 20))
-  (segment (start 122.047 65.532) (end 123.76625 67.25125) (width 0.254) (layer B.Cu) (net 70))
-  (segment (start 122.047 52.755) (end 122.047 65.532) (width 0.254) (layer B.Cu) (net 70))
-  (segment (start 123.76625 51.03575) (end 122.047 52.755) (width 0.254) (layer B.Cu) (net 70) (status 10))
-  (segment (start 123.76625 50.95875) (end 123.76625 51.03575) (width 0.254) (layer B.Cu) (net 70) (status 30))
   (segment (start 123.76625 86.11075) (end 123.76625 89.05875) (width 0.254) (layer B.Cu) (net 70) (status 20))
   (segment (start 122.047 84.3915) (end 123.76625 86.11075) (width 0.254) (layer B.Cu) (net 70))
@@
   (segment (start 133.29125 137.48225) (end 130.81 135.001) (width 0.254) (layer B.Cu) (net 70))
   (segment (start 133.29125 146.20875) (end 133.29125 137.48225) (width 0.254) (layer B.Cu) (net 70) (status 10))
+  (segment (start 123.444 69.6865) (end 123.76625 70.00875) (width 0.254) (layer B.Cu) (net 70))
+  (segment (start 123.444 67.056) (end 123.444 69.6865) (width 0.254) (layer B.Cu) (net 70))
+  (segment (start 122.047 65.659) (end 123.444 67.056) (width 0.254) (layer B.Cu) (net 70))
+  (segment (start 122.047 52.755) (end 122.047 65.659) (width 0.254) (layer B.Cu) (net 70))
+  (segment (start 123.76625 51.03575) (end 122.047 52.755) (width 0.254) (layer B.Cu) (net 70))
+  (segment (start 123.76625 50.95875) (end 123.76625 51.03575) (width 0.254) (layer B.Cu) (net 70))
   (segment (start 142.81625 89.05875) (end 142.81625 70.00875) (width 0.254) (layer B.Cu) (net 71) (status 30))
   (via (at 140.97 52.832106) (size 0.6) (drill 0.3) (layers F.Cu B.Cu) (net 71))
@@
   (segment (start 178.425 82.768) (end 177.1365 82.768) (width 0.254) (layer B.Cu) (net 79) (status 20))
   (segment (start 179.086 81.407) (end 179.086 82.107) (width 0.254) (layer B.Cu) (net 79) (status 10))
-  (segment (start 127.63125 62.64375) (end 127.79375 62.80625) (width 0.381) (layer B.Cu) (net 105) (status 30))
-  (segment (start 124.61875 62.64375) (end 127.63125 62.64375) (width 0.381) (layer B.Cu) (net 105) (status 30))
   (segment (start 128.259375 43.337153) (end 128.259375 44.129375) (width 0.381) (layer B.Cu) (net 105) (status 20))
   (segment (start 126.959222 42.037) (end 128.259375 43.337153) (width 0.381) (layer B.Cu) (net 105))
@@
   (segment (start 123.359375 43.328125) (end 124.6505 42.037) (width 0.381) (layer B.Cu) (net 105))
   (segment (start 123.359375 44.129375) (end 123.359375 43.328125) (width 0.381) (layer B.Cu) (net 105) (status 10))
-  (segment (start 122.682 61.688) (end 123.63775 62.64375) (width 0.381) (layer B.Cu) (net 105))
   (segment (start 122.682 56.7055) (end 122.682 61.688) (width 0.381) (layer B.Cu) (net 105))
   (segment (start 125.73 53.6575) (end 122.682 56.7055) (width 0.381) (layer B.Cu) (net 105))
@@
   (segment (start 123.359375 47.018671) (end 125.73 49.389296) (width 0.381) (layer B.Cu) (net 105))
   (segment (start 123.359375 44.129375) (end 123.359375 47.018671) (width 0.381) (layer B.Cu) (net 105) (status 10))
-  (segment (start 123.63775 62.64375) (end 124.61875 62.64375) (width 0.381) (layer B.Cu) (net 105) (status 20))
+  (segment (start 123.7685 62.7745) (end 124.587 62.7745) (width 0.381) (layer B.Cu) (net 105))
+  (segment (start 122.682 61.688) (end 123.7685 62.7745) (width 0.381) (layer B.Cu) (net 105))
   (segment (start 146.175 68.074) (end 146.177 68.072) (width 0.254) (layer B.Cu) (net 106))
   (segment (start 146.175 115.084618) (end 146.175 68.074) (width 0.254) (layer B.Cu) (net 106))
