File: tfk20-avr/tfk20-avr_rgb_matrix.sch (KiCad schematic (older format))
At the start: 34 parts, among them U2 IS31FL3733-TQ

Commit message: Assigned remaining footprints
Parts:
- D31, D32, D33, D34, D35, D36, D37, D38, D39, D40, D41, D42, D43, D44, D45, D46, D47, D48, D49, D50, D51: footprint (none) -> random-keyboard-parts:RGB-6028
Changed lines of the file:
@@
 F 0 "D31" H 1800 1500 50  0000 C CNN
 F 1 "LED_RGBA" H 1800 1506 50  0001 C CNN
-F 2 "" H 1800 1050 50  0001 C CNN
+F 2 "random-keyboard-parts:RGB-6028" H 1800 1050 50  0001 C CNN
 F 3 "~" H 1800 1050 50  0001 C CNN
 	1    1800 1100
@@
 F 0 "D32" H 2750 1500 50  0000 C CNN
 F 1 "LED_RGBA" H 2750 1506 50  0001 C CNN
-F 2 "" H 2750 1050 50  0001 C CNN
+F 2 "random-keyboard-parts:RGB-6028" H 2750 1050 50  0001 C CNN
 F 3 "~" H 2750 1050 50  0001 C CNN
 	1    2750 1100
@@
 F 0 "D33" H 3700 1500 50  0000 C CNN
 F 1 "LED_RGBA" H 3700 1506 50  0001 C CNN
-F 2 "" H 3700 1050 50  0001 C CNN
+F 2 "random-keyboard-parts:RGB-6028" H 3700 1050 50  0001 C CNN
 F 3 "~" H 3700 1050 50  0001 C CNN
 	1    3700 1100
@@
 F 0 "D35" H 1800 2700 50  0000 C CNN
 F 1 "LED_RGBA" H 1800 2706 50  0001 C CNN
-F 2 "" H 1800 2250 50  0001 C CNN
+F 2 "random-keyboard-parts:RGB-6028" H 1800 2250 50  0001 C CNN
 F 3 "~" H 1800 2250 50  0001 C CNN
 	1    1800 2300
@@
 F 0 "D36" H 2750 2700 50  0000 C CNN
 F 1 "LED_RGBA" H 2750 2706 50  0001 C CNN
-F 2 "" H 2750 2250 50  0001 C CNN
+F 2 "random-keyboard-parts:RGB-6028" H 2750 2250 50  0001 C CNN
 F 3 "~" H 2750 2250 50  0001 C CNN
 	1    2750 2300
@@
 F 0 "D37" H 3700 2700 50  0000 C CNN
 F 1 "LED_RGBA" H 3700 2706 50  0001 C CNN
-F 2 "" H 3700 2250 50  0001 C CNN
+F 2 "random-keyboard-parts:RGB-6028" H 3700 2250 50  0001 C CNN
 F 3 "~" H 3700 2250 50  0001 C CNN
 	1    3700 2300
@@
 F 0 "D34" H 4600 1500 50  0000 C CNN
 F 1 "LED_RGBA" H 4600 1506 50  0001 C CNN
-F 2 "" H 4600 1050 50  0001 C CNN
+F 2 "random-keyboard-parts:RGB-6028" H 4600 1050 50  0001 C CNN
 F 3 "~" H 4600 1050 50  0001 C CNN
 	1    4600 1100
@@
 F 0 "D38" H 4600 2700 50  0000 C CNN
 F 1 "LED_RGBA" H 4600 2706 50  0001 C CNN
-F 2 "" H 4600 2250 50  0001 C CNN
+F 2 "random-keyboard-parts:RGB-6028" H 4600 2250 50  0001 C CNN
 F 3 "~" H 4600 2250 50  0001 C CNN
 	1    4600 2300
@@
 F 0 "D39" H 1800 3900 50  0000 C CNN
 F 1 "LED_RGBA" H 1800 3906 50  0001 C CNN
-F 2 "" H 1800 3450 50  0001 C CNN
+F 2 "random-keyboard-parts:RGB-6028" H 1800 3450 50  0001 C CNN
 F 3 "~" H 1800 3450 50  0001 C CNN
 	1    1800 3500
@@
 F 0 "D40" H 2750 3900 50  0000 C CNN
 F 1 "LED_RGBA" H 2750 3906 50  0001 C CNN
-F 2 "" H 2750 3450 50  0001 C CNN
+F 2 "random-keyboard-parts:RGB-6028" H 2750 3450 50  0001 C CNN
 F 3 "~" H 2750 3450 50  0001 C CNN
 	1    2750 3500
@@
 F 0 "D41" H 3700 3900 50  0000 C CNN
 F 1 "LED_RGBA" H 3700 3906 50  0001 C CNN
-F 2 "" H 3700 3450 50  0001 C CNN
+F 2 "random-keyboard-parts:RGB-6028" H 3700 3450 50  0001 C CNN
 F 3 "~" H 3700 3450 50  0001 C CNN
 	1    3700 3500
@@
 F 0 "D42" H 1800 5100 50  0000 C CNN
 F 1 "LED_RGBA" H 1800 5106 50  0001 C CNN
-F 2 "" H 1800 4650 50  0001 C CNN
+F 2 "random-keyboard-parts:RGB-6028" H 1800 4650 50  0001 C CNN
 F 3 "~" H 1800 4650 50  0001 C CNN
 	1    1800 4700
@@
 F 0 "D43" H 2750 5100 50  0000 C CNN
 F 1 "LED_RGBA" H 2750 5106 50  0001 C CNN
-F 2 "" H 2750 4650 50  0001 C CNN
+F 2 "random-keyboard-parts:RGB-6028" H 2750 4650 50  0001 C CNN
 F 3 "~" H 2750 4650 50  0001 C CNN
 	1    2750 4700
@@
 F 0 "D44" H 3700 5100 50  0000 C CNN
 F 1 "LED_RGBA" H 3700 5106 50  0001 C CNN
-F 2 "" H 3700 4650 50  0001 C CNN
+F 2 "random-keyboard-parts:RGB-6028" H 3700 4650 50  0001 C CNN
 F 3 "~" H 3700 4650 50  0001 C CNN
 	1    3700 4700
@@
 F 0 "D45" H 4600 5100 50  0000 C CNN
 F 1 "LED_RGBA" H 4600 5106 50  0001 C CNN
-F 2 "" H 4600 4650 50  0001 C CNN
+F 2 "random-keyboard-parts:RGB-6028" H 4600 4650 50  0001 C CNN
 F 3 "~" H 4600 4650 50  0001 C CNN
 	1    4600 4700
@@
 F 0 "D46" H 1800 6300 50  0000 C CNN
 F 1 "LED_RGBA" H 1800 6306 50  0001 C CNN
-F 2 "" H 1800 5850 50  0001 C CNN
+F 2 "random-keyboard-parts:RGB-6028" H 1800 5850 50  0001 C CNN
 F 3 "~" H 1800 5850 50  0001 C CNN
 	1    1800 5900
@@
 F 0 "D47" H 2750 6300 50  0000 C CNN
 F 1 "LED_RGBA" H 2750 6306 50  0001 C CNN
-F 2 "" H 2750 5850 50  0001 C CNN
+F 2 "random-keyboard-parts:RGB-6028" H 2750 5850 50  0001 C CNN
 F 3 "~" H 2750 5850 50  0001 C CNN
 	1    2750 5900
@@
 F 0 "D48" H 3700 6300 50  0000 C CNN
 F 1 "LED_RGBA" H 3700 6306 50  0001 C CNN
-F 2 "" H 3700 5850 50  0001 C CNN
+F 2 "random-keyboard-parts:RGB-6028" H 3700 5850 50  0001 C CNN
 F 3 "~" H 3700 5850 50  0001 C CNN
 	1    3700 5900
@@
 F 0 "D51" H 4600 7500 50  0000 C CNN
 F 1 "LED_RGBA" H 4600 7506 50  0001 C CNN
-F 2 "" H 4600 7050 50  0001 C CNN
+F 2 "random-keyboard-parts:RGB-6028" H 4600 7050 50  0001 C CNN
 F 3 "~" H 4600 7050 50  0001 C CNN
 	1    4600 7100
@@
 F 0 "D50" H 3700 7500 50  0000 C CNN
 F 1 "LED_RGBA" H 3700 7506 50  0001 C CNN
-F 2 "" H 3700 7050 50  0001 C CNN
+F 2 "random-keyboard-parts:RGB-6028" H 3700 7050 50  0001 C CNN
 F 3 "~" H 3700 7050 50  0001 C CNN
 	1    3700 7100
@@
 F 0 "D49" H 1800 7500 50  0000 C CNN
 F 1 "LED_RGBA" H 1800 7506 50  0001 C CNN
-F 2 "" H 1800 7050 50  0001 C CNN
+F 2 "random-keyboard-parts:RGB-6028" H 1800 7050 50  0001 C CNN
 F 3 "~" H 1800 7050 50  0001 C CNN
 	1    1800 7100

Commit message: Begin PCB
Parts:
- R10, R11, R12, R13, R9: footprint Resistor_SMD:R_0815_2038Metric_Pad1.20x4.05mm_HandSolder -> Resistor_SMD:R_0805_2012Metric_Pad1.20x1.40mm_HandSolder
Changed lines of the file:
@@
 F 0 "R12" H 8091 2704 50  0000 R CNN
 F 1 "100k" H 8091 2795 50  0000 R CNN
-F 2 "Resistor_SMD:R_0815_2038Metric_Pad1.20x4.05mm_HandSolder" H 8150 2750 50  0001 C CNN
+F 2 "Resistor_SMD:R_0805_2012Metric_Pad1.20x1.40mm_HandSolder" H 8150 2750 50  0001 C CNN
 F 3 "~" H 8150 2750 50  0001 C CNN
 	1    8150 2750
@@
 F 0 "R9" H 7409 1996 50  0000 L CNN
 F 1 "100k" H 7409 1905 50  0000 L CNN
-F 2 "Resistor_SMD:R_0815_2038Metric_Pad1.20x4.05mm_HandSolder" H 7350 1950 50  0001 C CNN
+F 2 "Resistor_SMD:R_0805_2012Metric_Pad1.20x1.40mm_HandSolder" H 7350 1950 50  0001 C CNN
 F 3 "~" H 7350 1950 50  0001 C CNN
 	1    7350 1950
@@
 F 0 "R10" H 7809 1996 50  0000 L CNN
 F 1 "1k" H 7809 1905 50  0000 L CNN
-F 2 "Resistor_SMD:R_0815_2038Metric_Pad1.20x4.05mm_HandSolder" H 7750 1950 50  0001 C CNN
+F 2 "Resistor_SMD:R_0805_2012Metric_Pad1.20x1.40mm_HandSolder" H 7750 1950 50  0001 C CNN
 F 3 "~" H 7750 1950 50  0001 C CNN
 	1    7750 1950
@@
 F 0 "R11" H 8209 1996 50  0000 L CNN
 F 1 "1k" H 8209 1905 50  0000 L CNN
-F 2 "Resistor_SMD:R_0815_2038Metric_Pad1.20x4.05mm_HandSolder" H 8150 1950 50  0001 C CNN
+F 2 "Resistor_SMD:R_0805_2012Metric_Pad1.20x1.40mm_HandSolder" H 8150 1950 50  0001 C CNN
 F 3 "~" H 8150 1950 50  0001 C CNN
 	1    8150 1950
@@
 F 0 "R13" H 8791 3004 50  0000 R CNN
 F 1 "100k" H 8791 3095 50  0000 R CNN
-F 2 "Resistor_SMD:R_0815_2038Metric_Pad1.20x4.05mm_HandSolder" H 8850 3050 50  0001 C CNN
+F 2 "Resistor_SMD:R_0805_2012Metric_Pad1.20x1.40mm_HandSolder" H 8850 3050 50  0001 C CNN
 F 3 "~" H 8850 3050 50  0001 C CNN
 	1    8850 3050

Commit message: Continue routing
Connections:
- net SW1: now also U2.9 (SW7); no longer U2.2 (SW1)
- net SW2: now also U2.10 (SW8); no longer U2.3 (SW2)
- net SW3: now also U2.11 (SW9); no longer U2.4 (SW3)
- net SW7: now also U2.2 (SW1); no longer U2.9 (SW7)
- net SW8: now also U2.3 (SW2); no longer U2.10 (SW8)
- net SW9: now also U2.4 (SW3); no longer U2.11 (SW9)
Changed lines of the file:
@@
 Text Label 10750 2250 0    50   ~ 0
 CS4
-Text Label 10750 3650 0    50   ~ 0
+Text Label 10750 4250 0    50   ~ 0
 SW1
-Text Label 10750 3750 0    50   ~ 0
+Text Label 10750 4350 0    50   ~ 0
 SW2
-Text Label 10750 3850 0    50   ~ 0
+Text Label 10750 4450 0    50   ~ 0
 SW3
 Text Label 10750 3950 0    50   ~ 0
@@
 Text Label 10750 4150 0    50   ~ 0
 SW6
-Text Label 10750 4250 0    50   ~ 0
+Text Label 10750 3650 0    50   ~ 0
 SW7
-Text Label 10750 4350 0    50   ~ 0
+Text Label 10750 3750 0    50   ~ 0
 SW8
-Text Label 10750 4450 0    50   ~ 0
+Text Label 10750 3850 0    50   ~ 0
 SW9
 Wire Notes Line

Commit message: Clean up
Connections:
- net SW1: now also D46.3 (BK), D47.3 (BK), D48.3 (BK), D49.3 (BK), D50.3 (BK), D51.3 (BK), U2.2 (SW1); no longer D31.3 (BK), D32.3 (BK), D33.3 (BK), D34.3 (BK), D35.3 (BK), D36.3 (BK), D37.3 (BK), D38.3 (BK), U2.9 (SW7)
- net SW2: now also D46.1 (RK), D47.1 (RK), D48.1 (RK), D49.1 (RK), D50.1 (RK), D51.1 (RK), U2.3 (SW2); no longer D31.1 (RK), D32.1 (RK), D33.1 (RK), D34.1 (RK), D35.1 (RK), D36.1 (RK), D37.1 (RK), D38.1 (RK), U2.10 (SW8)
- net SW3: now also D46.2 (GK), D47.2 (GK), D48.2 (GK), D49.2 (GK), D50.2 (GK), D51.2 (GK), U2.4 (SW3); no longer D31.2 (GK), D32.2 (GK), D33.2 (GK), D34.2 (GK), D35.2 (GK), D36.2 (GK), D37.2 (GK), D38.2 (GK), U2.11 (SW9)
- net SW7: now also D31.3 (BK), D32.3 (BK), D33.3 (BK), D34.3 (BK), D35.3 (BK), D36.3 (BK), D37.3 (BK), D38.3 (BK), U2.9 (SW7); no longer D46.3 (BK), D47.3 (BK), D48.3 (BK), D49.3 (BK), D50.3 (BK), D51.3 (BK), U2.2 (SW1)
- net SW8: now also D31.1 (RK), D32.1 (RK), D33.1 (RK), D34.1 (RK), D35.1 (RK), D36.1 (RK), D37.1 (RK), D38.1 (RK), U2.10 (SW8); no longer D46.1 (RK), D47.1 (RK), D48.1 (RK), D49.1 (RK), D50.1 (RK), D51.1 (RK), U2.3 (SW2)
- net SW9: now also D31.2 (GK), D32.2 (GK), D33.2 (GK), D34.2 (GK), D35.2 (GK), D36.2 (GK), D37.2 (GK), D38.2 (GK), U2.11 (SW9); no longer D46.2 (GK), D47.2 (GK), D48.2 (GK), D49.2 (GK), D50.2 (GK), D51.2 (GK), U2.4 (SW3)
Changed lines of the file:
@@
 Text Label 10750 2250 0    50   ~ 0
 CS4
-Text Label 10750 4250 0    50   ~ 0
+Text Label 10750 3650 0    50   ~ 0
 SW1
-Text Label 10750 4350 0    50   ~ 0
+Text Label 10750 3750 0    50   ~ 0
 SW2
-Text Label 10750 4450 0    50   ~ 0
+Text Label 10750 3850 0    50   ~ 0
 SW3
 Text Label 10750 3950 0    50   ~ 0
@@
 Text Label 10750 4150 0    50   ~ 0
 SW6
-Text Label 10750 3650 0    50   ~ 0
+Text Label 10750 4250 0    50   ~ 0
 SW7
-Text Label 10750 3750 0    50   ~ 0
+Text Label 10750 4350 0    50   ~ 0
 SW8
-Text Label 10750 3850 0    50   ~ 0
+Text Label 10750 4450 0    50   ~ 0
 SW9
 Wire Notes Line
@@
 	2000 1100 2050 1100
 Wire Wire Line
-	850  1500 950  1500
-Wire Wire Line
 	1600 1300 1550 1300
 Wire Wire Line
@@
 Wire Wire Line
 	1600 1100 1450 1100
-Wire Wire Line
-	850  1700 1150 1700
-Wire Wire Line
-	850  1600 1050 1600
 Wire Wire Line
 	1450 1100 1450 1700
@@
 Text Label 4850 650  0    50   ~ 0
 CS4
-Text Label 850  1500 2    50   ~ 0
-SW1
-Text Label 850  1600 2    50   ~ 0
-SW2
-Text Label 850  1700 2    50   ~ 0
-SW3
 Text Label 850  3900 2    50   ~ 0
 SW4
@@
 Wire Wire Line
 	950  1500 950  2700
-Connection ~ 950  1500
 Wire Wire Line
 	950  1500 1550 1500
@@
 Wire Wire Line
 	1050 1600 1050 2800
-Connection ~ 1050 1600
 Wire Wire Line
 	1050 1600 1350 1600
@@
 Wire Wire Line
 	1150 1700 1150 2900
-Connection ~ 1150 1700
 Wire Wire Line
 	1150 1700 1450 1700
@@
 Wire Wire Line
 	1150 6500 850  6500
-Text Label 850  6300 2    50   ~ 0
+Text Label 850  1500 2    50   ~ 0
 SW7
-Text Label 850  6400 2    50   ~ 0
+Text Label 850  1600 2    50   ~ 0
 SW8
-Text Label 850  6500 2    50   ~ 0
+Text Label 850  1700 2    50   ~ 0
 SW9
 NoConn ~ 10700 4550
@@
 Wire Wire Line
 	1550 7500 3450 7500
+Connection ~ 1150 1700
+Connection ~ 1050 1600
+Connection ~ 950  1500
+Text Label 850  6500 2    50   ~ 0
+SW3
+Text Label 850  6400 2    50   ~ 0
+SW2
+Text Label 850  6300 2    50   ~ 0
+SW1
+Wire Wire Line
+	850  1600 1050 1600
+Wire Wire Line
+	850  1700 1150 1700
+Wire Wire Line
+	850  1500 950  1500
 $EndSCHEMATC
