File: tfk84-avr/tfk84-avr_rgb_light.sch (KiCad schematic (older format))
At the start: 24 parts

Commit message: Continue schematic
Parts:
- gave numbers to parts that had none: 12
- renumbered D25 to D4, D26 to D5, D27 to D6, D28 to D7, D29 to D8, D30 to D9
