File: tfk84-avr/tfk84-avr_rgb_matrix_m.sch (KiCad schematic (older format))
At the start: 42 parts

Commit message: Continue schematic
Parts:
- gave numbers to parts that had none: 42

Commit message: Begin PCB
Parts:
- D16, D17, D18, D19, D20, D21, D22, D23, D24, D25, D26, D27, D28, D29, D30, D31, D32, D33, D34, D35, D36, D37, D38, D39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: footprint (none) -> random-keyboard-parts:RGB-6028
Other:
- moved on the sheet: D16, D17, D18, D19, D20, D21, D22, D23, D24, D25, D26, D27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
