File: tfk84-avr/tfk84-avr_rgb_matrix_s.sch (KiCad schematic (older format))
At the start: 42 parts

Commit message: Continue schematic
Parts:
- gave numbers to parts that had none: 42

Commit message: Begin PCB
Parts:
- D58, D59, D60, D61, D62, D63, D64, D65, D66, D67, D68, D69, D70, D71, D72, D73, D74, D75, D76, D77, D78, D79, D80, D81, D82, D83, D84, D85, D86, D87, D88, D89, D90, D91, D92, D93, D94, D95, D96, D97, D98, D99: footprint (none) -> random-keyboard-parts:RGB-6028

Commit message: Continue layout
Connections:
- net S_CS1: now also D72.4 (A), D86.4 (A)
- net S_CS3: now also D73.4 (A), D87.4 (A)
- net S_SW3: now also D65.3 (BK), D66.3 (BK), D67.3 (BK), D68.3 (BK), D69.3 (BK), D70.3 (BK), D71.3 (BK)
Changed lines of the file:
@@
 	1000 1800 1200 1800
-Wire Wire Line
-	950  2850 950  2700
 Wire Wire Line
 	950  2850 1250 2850
@@
 	6800 2400 6950 2400
 Connection ~ 1800 1400
-Wire Wire Line
-	2650 1400 2650 1500
 Connection ~ 2650 1400
 Connection ~ 3500 1400
@@
 	6900 1400 6900 3400
 Connection ~ 6900 1400
-Wire Wire Line
-	1800 1400 1800 1500
 Wire Wire Line
 	1700 2400 1850 2400
@@
 	6950 600  6950 2400
 Wire Wire Line
-	1800 1900 1800 2500
-Wire Wire Line
-	2650 1900 2650 2500
-Wire Wire Line
-	950  2500 950  1850
-Wire Wire Line
-	1800 2900 1800 3400
-Wire Wire Line
-	2650 2900 2650 3400
-Wire Wire Line
 	1800 700  1800 1400
 Wire Wire Line
 	2650 700  2650 1400
+Wire Wire Line
+	950  1850 950  2850
+Wire Wire Line
+	2650 1400 2650 3400
+Wire Wire Line
+	1800 1400 1800 3400
 $EndSCHEMATC
