File: tfk84-avr/tfk84-avr_rgb_matrix.sch (KiCad schematic (older format))
At the start: 38 parts, among them U2 IS31FL3733B-TQLS4-TR

Commit message: Add RGB matrices
Parts:
- removed D31, D32, D33, D34, D35, D36, D37, D38, D39, D40, D41, D42, D43, D44, D45, D46, D47, D48, D49, D50, D51: LED_RGBA, random-keyboard-parts:RGB-6028, symbol Device:LED_RGBA
- added C? (x3): 470n, Capacitor_SMD:C_0805_2012Metric_Pad1.18x1.45mm_HandSolder, symbol Device:C
- added C? (x3): 100n, Capacitor_SMD:C_0805_2012Metric_Pad1.18x1.45mm_HandSolder, symbol Device:C
Connections:
- net labels removed: ADVCC, CS1, CS2, CS3, CS4, CS5, CS6, CS7, CS8, PVCC1, PVCC2, SW1, SW2, SW3, SW4, SW5, SW6, SW7, SW8, SW9
- wire segments 418 -> 196
- no-connect marks 24 -> 12
Other:
- note removed: "3 switches and\n8 current sources\nper 2 rows on pad"
- note removed: "Decoupling capacitors for LED driver"
- note removed: "RGB LED Matrix"
- moved on the sheet: C17, C18, C19, C20, C21, C22, C23, C?, R10, R11, R12, R13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

Commit message: Continue schematic
Parts:
- U2: symbol Driver_LED:IS31FL3733-TQ -> random-keyboard-parts:IS31FL3733B-TQ
- U3: renamed from U?; symbol Driver_LED:IS31FL3733-TQ -> random-keyboard-parts:IS31FL3733B-TQ
- gave numbers to parts that had none: 9
- renumbered C18 to C23, C19 to C24, C20 to C25, C21 to C26, C22 to C27, C23 to C28, C17 to C35, R12 to R13, R13 to R14

Commit message: Begin PCB
Other:
- note added: "I2C addresses"
- note added: "Master RGB LED driver"
- note added: "Slave RGB LED driver"
- moved on the sheet: C23, C24, C25, C26, C27, C28, C29, C30, C31, C32, C33, C34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
