File: tfk84-avr/tfk84-avr.kicad_pcb (KiCad board)
At the start: 4 copper layers, 304.8 x 114.3 mm, 346 parts, among them J1 USB_C_Receptacle_USB2.0, J2 AVR-ISP-6, SW1 Reset, U1 ATmega32U4-AU, U2 IS31FL3733B-TQLS4-TR, U3 IS31FL3733B-TQLS4-TR, Y1 16MHz

Commit message: Layout backlight LEDs
Parts:
- C13, C14, C15, C16, C17, C18, C19, C20, C21, C22: moved to B.Cu
- moved C13 523.4 mm to (78.6, 185.2)
- moved C14 495.7 mm to (77.4, 108.3)
- moved C15 426.1 mm to (134.5, 108.3)
- moved C16 396.3 mm to (191.7, 108.3)
- moved C22 396.1 mm to (233.4, 187.3)
- moved C17 354.3 mm to (229.8, 108.3)
- moved C21 339.8 mm to (283.8, 182.2), turned to 90 degrees
- moved C20 281.9 mm to (344.5, 187.3)
- moved C18 276.7 mm to (286.9, 108.3)
- moved C19 233.5 mm to (344.1, 108.3)
- moved D15 174.8 mm to (234.9, 183.4)
- moved D7 173.8 mm to (79.0, 104.4), turned to 0 degrees
- moved D13 171.6 mm to (345.7, 183.4)
- moved D9 171.6 mm to (193.3, 104.4), turned to 0 degrees
- moved D14 171.6 mm to (288.5, 183.4)
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
Commit message: Place all components on board
Parts:
- moved R14 63.9 mm to (211.2, 179.3), turned to 270 degrees
- moved R11 41.0 mm to (175.5, 194.3), turned to 180 degrees
- moved R13 40.8 mm to (213.9, 193.7), turned to 90 degrees
- moved R12 40.6 mm to (217.2, 181.4), turned to 270 degrees
- moved R15 40.6 mm to (220.0, 193.7), turned to 90 degrees
- moved R10 40.2 mm to (175.5, 191.6), turned to 180 degrees
- moved C27 39.1 mm to (214.2, 180.2)
- moved C28 39.1 mm to (214.2, 182.2)
- moved C35 39.1 mm to (214.2, 178.2)
- moved C34 33.7 mm to (216.9, 190.7)
- moved C33 30.0 mm to (216.9, 192.7), turned to 180 degrees
- moved C26 27.8 mm to (204.1, 180.7), turned to 90 degrees
- moved C25 27.5 mm to (202.1, 180.7), turned to 90 degrees
- moved C36 26.3 mm to (216.9, 194.7), turned to 180 degrees
- moved R9 26.3 mm to (211.8, 193.7)
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
Commit message: Layout switch diodes
Parts:
- added G***: LOGO, biosmanager:biosmanager_pcb, F.Cu at (159.1, 187.3)
- MX10, MX17, MX19, MX38, MX53, MX55, MX62, MX71: footprint Switch_Keyboard_Kailh:SW_Hotswap_Kailh_1.00u_NoFrontSilk -> Switch_Keyboard_Kailh:SW_Hotswap_Kailh_1.00u_NoFrontSilk_CornerPad
- MX13: footprint Switch_Keyboard_Kailh:SW_Hotswap_Kailh_1.50u -> Switch_Keyboard_Kailh:SW_Hotswap_Kailh_1.50u_NoFrontSilk_CornerPad
- MX14: footprint random-keyboard-parts:SW_Hotswap_Kailh_1.00u_NoFrontSilk_CornerPad_TightCrtYd -> Switch_Keyboard_Kailh:SW_Hotswap_Kailh_1.00u_NoFrontSilk_CornerPad
- MX23: footprint Switch_Keyboard_Kailh:SW_Hotswap_Kailh_1.50u -> Switch_Keyboard_Kailh:SW_Hotswap_Kailh_1.50u_NoFrontSilk
- MX25, MX59: footprint Switch_Keyboard_Kailh:SW_Hotswap_Kailh_1.75u -> Switch_Keyboard_Kailh:SW_Hotswap_Kailh_1.75u_NoFrontSilk
- MX35, MX37: footprint Switch_Keyboard_Kailh:SW_Hotswap_Kailh_2.25u -> Switch_Keyboard_Kailh:SW_Hotswap_Kailh_2.25u_NoFrontSilk
- MX49, MX61, MX73: footprint Switch_Keyboard_Kailh:SW_Hotswap_Kailh_1.25u -> Switch_Keyboard_Kailh:SW_Hotswap_Kailh_1.25u_NoFrontSilk
- MX77: footprint Switch_Keyboard_Kailh:SW_Hotswap_Kailh_6.25u -> Switch_Keyboard_Kailh:SW_Hotswap_Kailh_6.25u_NoFrontSilk
- moved C20 6.09 mm to (341.1, 182.2), turned to 90 degrees
- moved C7 2.45 mm to (156.4, 176.4), turned to 0 degrees
- moved C5 2.37 mm to (145.7, 179.8)
- moved D113 1.19 mm to (83.7, 100.4)
- moved C1 1.13 mm to (145.7, 181.9)
- moved D110 0.40 mm to (331.4, 100.4), turned to 180 degrees
- moved D148 0.40 mm to (63.1, 192.1)
- moved D160 0.40 mm to (86.9, 192.1)
- moved D170 0.40 mm to (308.4, 192.1)
- moved D172 0.40 mm to (110.7, 192.1)
- moved D176 0.40 mm to (182.2, 192.1)
- moved D180 0.40 mm to (251.2, 192.1)
- moved D181 0.40 mm to (270.3, 192.1)
- moved D182 0.40 mm to (289.3, 192.1)
- moved D183 0.40 mm to (327.4, 192.1)
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Other:
- outline, holes or cut-outs redrawn
- board text added: "Designed by biosmanager"
- board text added: "tfk84-avr"

Commit message: Minor tweaks
Parts:
- moved C14 5.68 mm to (74.4, 103.5), turned to 90 degrees
- moved C21 0.39 mm to (284.0, 182.5)
- moved C12 0.38 mm to (129.2, 182.5), turned to 90 degrees
- moved C20 0.25 mm to (341.1, 182.5)
Routing:
- net +5V: track 6.45 -> 60.8 mm, vias 2 -> 16
- net GND: track 3.71 -> 50.0 mm, vias 1 -> 30
- net VBUS: track 26.9 -> 34.5 mm
- net Net-(J1-PadB5): track 0.00 -> 6.69 mm, vias 0 -> 2
- net /RGB_MATRIX_SCL: track 0.00 -> 4.55 mm, vias 0 -> 1
- net /tfk84 RGB Matrix/SYNC: track 0.00 -> 4.52 mm, vias 0 -> 1
- net /IN_USB_D+: track 0.00 -> 4.48 mm
- net /tfk84 RGB Matrix/IICRST: track 0.00 -> 4.44 mm, vias 0 -> 1
- net /RGB_MATRIX_SDA: track 0.00 -> 4.42 mm, vias 0 -> 1
- net Net-(J1-PadA5): track 0.00 -> 4.35 mm
- net /IN_USB_D-: track 0.00 -> 2.96 mm
