File: tfk21-avr/tfk21-avr.kicad_pcb (KiCad board)
At the start: 4 copper layers, 76.2 x 115.5 mm, 123 parts, among them J1 USB_C_Receptacle_USB2.0, J2 AVR-ISP-6, SW1 Reset, U1 ATmega32U4-AU, U2 IS31FL3733-TQ, Y1 16MHz

Commit message: Fix LED driver resistors and mounting hole pads
Parts:
- R10, R11: value 1k -> 2k
- R13: value 100k -> 20k

Commit message: Tweak some things
Routing:
- net +5V: track 109.4 -> 110.7 mm, vias 15 -> 16
Changed lines of the file:
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@@
   (general
     (thickness 1.6)
-    (drawings 37)
-    (tracks 1695)
+    (drawings 38)
+    (tracks 1696)
     (zones 0)
     (modules 123)
@@
     (34 B.Paste user)
     (35 F.Paste user)
-    (36 B.SilkS user hide)
-    (37 F.SilkS user hide)
+    (36 B.SilkS user)
+    (37 F.SilkS user)
     (38 B.Mask user)
     (39 F.Mask user)
     (40 Dwgs.User user)
     (41 Cmts.User user)
-    (42 Eco1.User user hide)
-    (43 Eco2.User user hide)
+    (42 Eco1.User user)
+    (43 Eco2.User user)
     (44 Edge.Cuts user)
     (45 Margin user)
-    (46 B.CrtYd user hide)
-    (47 F.CrtYd user hide)
-    (48 B.Fab user hide)
-    (49 F.Fab user hide)
+    (46 B.CrtYd user)
+    (47 F.CrtYd user)
+    (48 B.Fab user)
+    (49 F.Fab user)
   )
   (setup
@@
     (tags "capacitor handsolder")
     (attr smd)
-    (fp_text reference C14 (at 0 -1.778 90) (layer B.SilkS)
+    (fp_text reference C14 (at 0 -2.413 180) (layer B.SilkS)
       (effects (font (size 1 1) (thickness 0.15)) (justify mirror))
     )
@@
     (tags "capacitor handsolder")
     (attr smd)
-    (fp_text reference C13 (at 0 -1.778 90) (layer B.SilkS)
+    (fp_text reference C13 (at 0 -2.413 180) (layer B.SilkS)
       (effects (font (size 1 1) (thickness 0.15)) (justify mirror))
     )
@@
     (tags "capacitor handsolder")
     (attr smd)
-    (fp_text reference C12 (at 0 -1.651 90) (layer B.SilkS)
+    (fp_text reference C12 (at -1.016 -2.286 180) (layer B.SilkS)
       (effects (font (size 1 1) (thickness 0.15)) (justify mirror))
     )
@@
     (tags "resistor handsolder")
     (attr smd)
-    (fp_text reference R8 (at 0 -1.651 270) (layer B.SilkS)
+    (fp_text reference R8 (at 0 -2.032) (layer B.SilkS)
       (effects (font (size 1 1) (thickness 0.15)) (justify mirror))
     )
@@
     (tags "resistor handsolder")
     (attr smd)
-    (fp_text reference R6 (at 0 1.65 90) (layer B.SilkS)
+    (fp_text reference R6 (at 0 1.905 180) (layer B.SilkS)
       (effects (font (size 1 1) (thickness 0.15)) (justify mirror))
     )
@@
     (tags "resistor handsolder")
     (attr smd)
-    (fp_text reference R5 (at 0 -1.68275 270) (layer B.SilkS)
+    (fp_text reference R5 (at 0 -1.905) (layer B.SilkS)
       (effects (font (size 1 1) (thickness 0.15)) (justify mirror))
     )
@@
     (tags "resistor handsolder")
     (attr smd)
-    (fp_text reference R4 (at 3.01625 0.03175 90) (layer B.SilkS)
+    (fp_text reference R4 (at 3.175 -0.127 180) (layer B.SilkS)
       (effects (font (size 1 1) (thickness 0.15)) (justify mirror))
     )
@@
       (effects (font (size 1 1) (thickness 0.15)))
     )
-    (fp_text value Case (at 0 3.5) (layer F.Fab)
-      (effects (font (size 1 1) (thickness 0.15)))
+    (fp_text value Case (at 0 3.96875) (layer B.SilkS)
+      (effects (font (size 1 1) (thickness 0.15)) (justify mirror))
     )
     (fp_circle (center 0 0) (end 2.75 0) (layer F.CrtYd) (width 0.05))
@@
     (tags "fuse handsolder")
     (attr smd)
-    (fp_text reference F1 (at 0 -1.778 90) (layer B.SilkS)
+    (fp_text reference F1 (at 0 -2.032 180) (layer B.SilkS)
       (effects (font (size 1 1) (thickness 0.15)) (justify mirror))
     )
@@
     (tags SOD-123)
     (attr smd)
-    (fp_text reference D23 (at 0 2 90) (layer B.SilkS)
+    (fp_text reference D23 (at -3.175 0 180) (layer B.SilkS)
       (effects (font (size 1 1) (thickness 0.15)) (justify mirror))
     )
@@
     (tags SOD-123)
     (attr smd)
-    (fp_text reference D22 (at 0 2 90) (layer B.SilkS)
+    (fp_text reference D22 (at 0 2.667 180) (layer B.SilkS)
       (effects (font (size 1 1) (thickness 0.15)) (justify mirror))
     )
@@
     (tags SOD-123)
     (attr smd)
-    (fp_text reference D11 (at 3.90525 0 90) (layer B.SilkS)
+    (fp_text reference D11 (at 3.175 0 180) (layer B.SilkS)
       (effects (font (size 1 1) (thickness 0.15)) (justify mirror))
     )
@@
     (tags SOD-123)
     (attr smd)
-    (fp_text reference D3 (at 0 1.74625 270) (layer B.SilkS)
+    (fp_text reference D3 (at 0 2.159) (layer B.SilkS)
       (effects (font (size 1 1) (thickness 0.15)) (justify mirror))
     )
@@
     (tags SOT-143)
     (attr smd)
-    (fp_text reference D2 (at 0.02 2.38) (layer B.SilkS)
+    (fp_text reference D2 (at 0.02 -2.54) (layer B.SilkS)
       (effects (font (size 1 1) (thickness 0.15)) (justify mirror))
     )
@@
     (tags SOD-123)
     (attr smd)
-    (fp_text reference D1 (at 0 2.032 90) (layer B.SilkS)
+    (fp_text reference D1 (at 0 2.286 180) (layer B.SilkS)
       (effects (font (size 1 1) (thickness 0.15)) (justify mirror))
     )
@@
     (tags "capacitor handsolder")
     (attr smd)
-    (fp_text reference C20 (at 0.127 -1.524) (layer B.SilkS)
+    (fp_text reference C20 (at -0.889 -1.524) (layer B.SilkS)
       (effects (font (size 1 1) (thickness 0.15)) (justify mirror))
     )
@@
     (tags "capacitor handsolder")
     (attr smd)
-    (fp_text reference C19 (at 0.5334 -2.413 270) (layer B.SilkS)
+    (fp_text reference C19 (at 0.9144 -1.524) (layer B.SilkS)
       (effects (font (size 1 1) (thickness 0.15)) (justify mirror))
     )
@@
     (tags "capacitor handsolder")
     (attr smd)
-    (fp_text reference C8 (at 0 1.778 270) (layer B.SilkS)
+    (fp_text reference C8 (at 0 2.032) (layer B.SilkS)
       (effects (font (size 1 1) (thickness 0.15)) (justify mirror))
     )
@@
     (tags "capacitor handsolder")
     (attr smd)
-    (fp_text reference C6 (at 3.175 0 90) (layer B.SilkS)
+    (fp_text reference C6 (at 3.175 0.127 180) (layer B.SilkS)
       (effects (font (size 1 1) (thickness 0.15)) (justify mirror))
     )
@@
     )
   )
+  (dimension 1.190625 (width 0.15) (layer Dwgs.User)
+    (gr_text "1.191 mm" (at 93 38.298437) (layer Dwgs.User)
+      (effects (font (size 1 1) (thickness 0.15)) (justify right))
+    )
+    (feature1 (pts (xy 120.253125 37.703125) (xy 93.869829 37.703125)))
+    (feature2 (pts (xy 120.253125 38.89375) (xy 93.869829 38.89375)))
+    (crossbar (pts (xy 94.45625 38.89375) (xy 94.45625 37.703125)))
+    (arrow1a (pts (xy 94.45625 37.703125) (xy 95.042671 38.829629)))
+    (arrow1b (pts (xy 94.45625 37.703125) (xy 93.869829 38.829629)))
+    (arrow2a (pts (xy 94.45625 38.89375) (xy 95.042671 37.767246)))
+    (arrow2b (pts (xy 94.45625 38.89375) (xy 93.869829 37.767246)))
+  )
   (dimension 2.5 (width 0.1) (layer Dwgs.User)
     (gr_text "2.500 mm" (at 84.13 57.94) (layer Dwgs.User)
@@
   (segment (start 161.8195 122.1525) (end 160.782 123.19) (width 0.381) (layer B.Cu) (net 1) (status 10))
   (segment (start 161.925 122.1525) (end 161.8195 122.1525) (width 0.381) (layer B.Cu) (net 1) (status 30))
-  (via (at 124.61875 67.157606) (size 0.8) (drill 0.4) (layers F.Cu B.Cu) (net 2))
   (via (at 147.0152 62.5348) (size 0.8) (drill 0.4) (layers F.Cu B.Cu) (net 2))
   (segment (start 147.023 62.527) (end 147.0152 62.5348) (width 0.381) (layer B.Cu) (net 2))
@@
   (segment (start 165.086055 87.503) (end 165.028795 87.56026) (width 0.381) (layer B.Cu) (net 2))
   (segment (start 166.386 87.503) (end 165.086055 87.503) (width 0.381) (layer B.Cu) (net 2) (status 10))
-  (segment (start 124.587 67.125856) (end 124.61875 67.157606) (width 0.381) (layer B.Cu) (net 2))
   (segment (start 124.6245 65.7495) (end 124.587 65.7495) (width 0.381) (layer B.Cu) (net 2) (status 30))
   (segment (start 124.7495 65.912) (end 124.587 65.7495) (width 0.381) (layer B.Cu) (net 2) (status 30))
   (segment (start 127.762 65.912) (end 124.7495 65.912) (width 0.381) (layer B.Cu) (net 2) (status 30))
   (segment (start 124.61875 65.78125) (end 124.587 65.7495) (width 0.381) (layer B.Cu) (net 2) (status 30))
-  (segment (start 124.61875 67.157606) (end 124.61875 65.78125) (width 0.381) (layer B.Cu) (net 2) (status 20))
   (segment (start 166.9542 74.9593) (end 166.9542 74.9554) (width 0.381) (layer B.Cu) (net 2))
   (segment (start 168.3219 76.327) (end 166.9542 74.9593) (width 0.381) (layer B.Cu) (net 2) (status 10))
@@
   (segment (start 162.0305 124.2275) (end 163.068 123.19) (width 0.381) (layer B.Cu) (net 2) (status 10))
   (segment (start 161.925 124.2275) (end 162.0305 124.2275) (width 0.381) (layer B.Cu) (net 2) (status 30))
+  (via (at 127.762 67.183) (size 0.8) (drill 0.4) (layers F.Cu B.Cu) (net 2))
+  (segment (start 127.762 65.912) (end 127.762 67.183) (width 0.381) (layer B.Cu) (net 2) (status 10))
+  (via (at 124.587 67.183) (size 0.8) (drill 0.4) (layers F.Cu B.Cu) (net 2))
+  (segment (start 124.587 65.7495) (end 124.587 67.183) (width 0.381) (layer B.Cu) (net 2) (status 10))
   (segment (start 130.129375 39.034375) (end 130.129375 43.214375) (width 0.254) (layer B.Cu) (net 3) (status 30))
   (segment (start 130.129375 39.034375) (end 121.489375 39.034375) (width 0.254) (layer B.Cu) (net 3) (status 30))
