File: tfk21-avr/tfk21-avr.kicad_pcb (KiCad board)
At the start: 4 copper layers, 76.2 x 115.5 mm, 123 parts, among them J1 USB_C_Receptacle_USB2.0, J2 AVR-ISP-6, SW1 Reset, U1 ATmega32U4-AU, U2 IS31FL3733-TQ, Y1 16MHz

Commit message: Tweak component values
Parts:
- C11, C12, C13, C14, C15, C16: value 104 -> 100n
- D1: value 5.5V -> 6V
- U2: value IS31FL3733-TQ -> IS31FL3733B-TQLS4-TR
