File: tfk21-avr/tfk21-avr.sch (KiCad schematic (older format))
At the start: 31 parts, among them J1 USB_C_Receptacle_USB2.0, J2 AVR-ISP-6, SW1 Reset, U1 ATmega32U4-AU, Y1 16MHz

Commit message: Rename tfk20 to tfk21
Changed lines of the file:
@@
 encoding utf-8
 Sheet 1 4
-Title "tfk20 AVR"
+Title "tfk21 AVR"
 Date "2021-02-02"
 Rev "0"
@@
 S 3550 4150 550  1200
 U 601C3315
-F0 "tfk20 Key Matrix" 50
-F1 "tfk20-avr_key_matrix.sch" 50
+F0 "tfk21 Key Matrix" 50
+F1 "tfk21-avr_key_matrix.sch" 50
 F2 "COL_0" I L 3550 4250 50
 F3 "COL_1" I L 3550 4350 50
@@
 S 5200 5050 600  200
 U 602C340B
-F0 "tfk20 RGB Light" 50
-F1 "tfk20-avr_rgb_light.sch" 50
+F0 "tfk21 RGB Light" 50
+F1 "tfk21-avr_rgb_light.sch" 50
 F2 "RGB_LIGHT" I L 5200 5150 50
 $EndSheet
@@
 S 5200 4150 600  300
 U 601F4644
-F0 "tfk20 RGB Matrix" 50
-F1 "tfk20-avr_rgb_matrix.sch" 50
+F0 "tfk21 RGB Matrix" 50
+F1 "tfk21-avr_rgb_matrix.sch" 50
 F2 "SDA" B L 5200 4350 50
 F3 "SCL" I L 5200 4250 50

Commit message: Tweak component values
Parts:
- D1: value 5.5V -> 6V
Changed lines of the file:
@@
 P 4000 1250
 F 0 "D1" V 3954 1320 50  0000 L CNN
-F 1 "5.5V" V 4045 1320 50  0000 L CNN
+F 1 "6V" V 4045 1320 50  0000 L CNN
 F 2 "Diode_SMD:D_SOD-123" V 4000 1250 50  0001 C CNN
 F 3 "~" V 4000 1250 50  0001 C CNN
